Commit message: add a can on top of the base_link

File: src/bot_description/urdf/bot.urdf.xacro (robot description, xacro)
@@ -69,3 +69,16 @@
         <origin xyz="-0.04755 0 -0.0275" rpy="0 0 0"/>
     </joint>
+    <link name="can_link" >
+        <visual>
+            <origin xyz="-0.03 0.03 0" rpy="1.57 0 0" />
+            <geometry>
+                <mesh filename="package://bot_description/meshes/can.STL"/>
+            </geometry>
+        </visual>
+    </link>
+    <joint name="can_joint" type="fixed">
+        <parent link="base_link"/>
+        <child link="can_link"/>
+        <origin xyz="0 0 0.078" rpy="0 0 0"/>
+    </joint>
 </robot>
